Commit message: added slam yaml file to perfrom online_async localizations and mapping.

File: mircobot_description/urdf/mircobot.xacro (robot description, xacro)
@@ -20,4 +20,12 @@
     </geometry>
   </collision>
+</link>
+    <!-- BASE_FOOTPRINT LINK -->
+<joint name="base_footprint_joint" type="fixed">
+    <parent link="base_link"/>
+    <child link="base_footprint"/>
+    <origin xyz="0 0 0" rpy="0 0 0"/>
+</joint>
+<link name="base_footprint">
 </link>
 <joint name="wheel_front_left_joint" type="fixed">

File: mircobot_description/urdf/mircobot_gazebo.xacro (robot description, xacro)
@@ -13,7 +13,7 @@
 <gazebo reference="wheel_back_left_1">
   <material>Gazebo/Black</material>
-  <!-- <mu1 value="0.6"/>
-  <mu2 value="0.6"/>
-  <self_collide>true</self_collide> -->
+  <mu1 value="0.5"/>
+  <mu2 value="0.5"/>
+  <self_collide>true</self_collide>
 </gazebo>
 <gazebo reference="wheel_front_right_1">
@@ -25,7 +25,7 @@
 <gazebo reference="wheel_back_right_1">
   <material>Gazebo/Black</material>
-  <!-- <mu1 value="0.6"/>
-  <mu2 value="0.6"/>
-  <self_collide>true</self_collide> -->
+   <mu1 value="0.5"/>
+  <mu2 value="0.5"/>
+  <self_collide>true</self_collide>
 </gazebo>
 <gazebo reference="lidar_1">
