Commit message: changed code for new gazebo

File: mircobot_description/urdf/materials.xacro (robot description, xacro)
@@ -4,3 +4,12 @@
     <color rgba="0.700 0.700 0.700 1.000"/>
   </material>
+  <material name="red">
+    <color rgba="1.000 0.000 0.000 1.000"/>
+  </material>
+  <material name="black">
+    <color rgba="0.000 0.000 0.000 1.000"/>
+  </material>
+  <material name="white">
+    <color rgba="1.000 1.000 1.000 1.000"/>
+  </material>
 </robot>

File: mircobot_description/urdf/mircobot_gazebo.xacro (robot description, xacro)
@@ -31,11 +31,12 @@
 <gazebo reference="lidar_1">
   <material>Gazebo/Black</material>
-  <sensor name="laser" type="ray">
+  <sensor name="laser" type="gpu_lidar">
+    <material>Gazebo/Black</material>
       <pose> 0 0 0 0 0 0 </pose>
-      <visualize>true</visualize>
-      <always_on>true</always_on>
-      <enable_processing>true</enable_processing>
+      <visualize>false</visualize>
+      <!-- <always_on>true</always_on> -->
+      <!-- <enable_processing>true</enable_processing> -->
       <update_rate>10</update_rate>
-      <ray>
+      <lidar>
           <scan>
               <horizontal>
@@ -49,15 +50,11 @@
               <max>12</max>
           </range>
-      </ray>
-      <plugin name="laser_controller" filename="libgazebo_ros_ray_sensor.so">
-        <ros>
-          <argument>~/out:=scan</argument>
-      </ros>
-      <output_type>sensor_msgs/LaserScan</output_type>
-      <frame_name>lidar_1</frame_name>
-      </plugin>
+      </lidar>
+          <topic>scan</topic>
+          <gz_frame_id>laser_frame</gz_frame_id>
   </sensor>
 </gazebo>
 <gazebo reference="camera_1">
+  <material>Gazebo/Black</material>
     <sensor type="camera" name="camera">
         <pose> 0 0 0 0 0 0 </pose>
@@ -65,4 +62,5 @@
         <update_rate>30.0</update_rate>
         <camera name="head">
+          <camera_info_topic>camera/camera_info</camera_info_topic>
           <horizontal_fov>1.089</horizontal_fov>
           <image>
@@ -76,12 +74,6 @@
           </clip>
         </camera>
-        <plugin name="camera_controller" filename="libgazebo_ros_camera.so">
-          <!-- <alwaysOn>true</alwaysOn>
-          <update_rate>0.0</update_rate> -->
-          <!-- <cameraName>mircobot/camera_optical</cameraName>
-          <imageTopicName>image_raw</imageTopicName>
-          <cameraInfoTopicName>camera_info</cameraInfoTopicName> -->
-          <frame_name>camera_optical</frame_name>
-        </plugin>
+        <topic>camera/image_raw</topic>
+        <gz_frame_id>camera_optical</gz_frame_id>
     </sensor>
 </gazebo>

File: mircobot_description/urdf/ros2_control.xacro (robot description, xacro)
@@ -3,5 +3,5 @@
     <ros2_control name="GazeboSystem" type="system">
         <hardware>
-            <plugin>gazebo_ros2_control/GazeboSystem</plugin>
+            <plugin>gz_ros2_control/GazeboSimSystem</plugin>
         </hardware>
         <!-- <joint name="wheel_front_left_joint">
@@ -39,6 +39,7 @@
     </ros2_control>
     <gazebo>
-        <plugin name="gazebo_ros2_control" filename="libgazebo_ros2_control.so">
+        <plugin name="gz_ros2_control::GazeboSimROS2ControlPlugin" filename="libgz_ros2_control-system.so">
             <parameters>$(find mircobot_description)/config/my_controllers.yaml</parameters>
+            <parameters>$(find mircobot_description)/config/gaz_ros2_ctl_use_sim.yaml</parameters>
         </plugin>
     </gazebo>
