Commit message: correct the ros2 control for 4 wheel drive, and changed it for new gazebo

File: mircobot_description/urdf/gazebo_control.xacro (robot description, xacro)
@@ -2,5 +2,5 @@
 <robot name="mircobot" xmlns:xacro="http://www.ros.org/wiki/xacro">
     <gazebo>
-        <plugin name='diff_drive' filename='libgazebo_ros_diff_drive.so'>
+        <plugin name="gz::sim::systems::DiffDrive" filename="gz-sim-diff-drive-system">
             <!-- Wheel Information -->
             <left_joint>wheel_back_left_joint</left_joint>
@@ -20,4 +20,10 @@
             <publish_wheel_tf>true</publish_wheel_tf>
         </plugin>
+        <plugin filename="gz-sim-joint-state-publisher-system"
+            name="gz::sim::systems::JointStatePublisher">
+            <topic>joint_states</topic>
+            <joint_name>wheel_back_left_joint</joint_name>
+            <joint_name>wheel_back_right_joint</joint_name>
+        </plugin>
     </gazebo>
 </robot>

File: mircobot_description/urdf/materials.xacro (robot description, xacro)
@@ -4,3 +4,12 @@
     <color rgba="0.700 0.700 0.700 1.000"/>
   </material>
+  <material name="red">
+    <color rgba="1.000 0.000 0.000 1.000"/>
+  </material>
+  <material name="black">
+    <color rgba="0.000 0.000 0.000 1.000"/>
+  </material>
+  <material name="white">
+    <color rgba="1.000 1.000 1.000 1.000"/>
+  </material>
 </robot>

File: mircobot_description/urdf/mircobot.xacro (robot description, xacro)
@@ -12,5 +12,5 @@
       <mesh filename="file://$(find mircobot_description)/meshes/base_link.stl" scale="0.001 0.001 0.001"/>
     </geometry>
-    <material name="silver"/>
+    <material name="red"/>
   </visual>
   <collision>
@@ -29,5 +29,5 @@
 <link name="base_footprint">
 </link>
-<joint name="wheel_front_left_joint" type="fixed">
+<joint name="wheel_front_left_joint" type="continuous">
   <origin xyz="0.05 0.065 0.025" rpy="-1.5708 0 0"/>
   <parent link="base_link"/>
@@ -46,5 +46,5 @@
       <mesh filename="file://$(find mircobot_description)/meshes/wheel_front_left_1.stl" scale="0.001 0.001 0.001"/>
     </geometry>
-    <material name="silver"/>
+    <material name="black"/>
   </visual>
   <collision>
@@ -72,5 +72,5 @@
       <mesh filename="file://$(find mircobot_description)/meshes/wheel_back_left_1.stl" scale="0.001 0.001 0.001"/>
     </geometry>
-    <material name="silver"/>
+    <material name="black"/>
   </visual>
   <collision>
@@ -81,5 +81,5 @@
   </collision>
 </link>
-<joint name="wheel_front_right_joint" type="fixed">
+<joint name="wheel_front_right_joint" type="continuous">
   <origin xyz="0.05 -0.065 0.025" rpy="-1.5708 0 0"/>
   <parent link="base_link"/>
@@ -98,5 +98,5 @@
       <mesh filename="file://$(find mircobot_description)/meshes/wheel_front_right_1.stl" scale="0.001 0.001 0.001"/>
     </geometry>
-    <material name="silver"/>
+    <material name="black"/>
   </visual>
   <collision>
@@ -124,5 +124,5 @@
       <mesh filename="file://$(find mircobot_description)/meshes/wheel_back_right_1.stl" scale="0.001 0.001 0.001"/>
     </geometry>
-    <material name="silver"/>
+    <material name="black"/>
   </visual>
   <collision>
@@ -136,7 +136,7 @@
   <origin xyz="0.0 0.0 0.06" rpy="0 0 0"/>
   <parent link="base_link"/>
-  <child link="lidar_1"/>
+  <child link="lidar"/>
 </joint>
-<link name="lidar_1">
+<link name="lidar">
   <inertial>
     <origin xyz="-1.7763568394002505e-17 -7.385233546074017e-18 0.010000000000000009" rpy="0 0 0"/>
@@ -149,5 +149,5 @@
       <mesh filename="file://$(find mircobot_description)/meshes/lidar_1.stl" scale="0.001 0.001 0.001"/>
     </geometry>
-    <material name="silver"/>
+    <material name="black"/>
   </visual>
   <collision>

File: mircobot_description/urdf/mircobot_gazebo.xacro (robot description, xacro)
@@ -7,6 +7,6 @@
 <gazebo reference="wheel_front_left_1">
   <material>Gazebo/Black</material>
-  <mu1 value="0.01"/>
-  <mu2 value="0.01"/>
+  <mu1 value="0.5"/>
+  <mu2 value="0.5"/>
   <!-- <self_collide>true</self_collide> -->
 </gazebo>
@@ -19,6 +19,6 @@
 <gazebo reference="wheel_front_right_1">
   <material>Gazebo/Black</material>
-  <mu1 value="0.01"/>
-  <mu2 value="0.01"/>
+  <mu1 value="0.5"/>
+  <mu2 value="0.5"/>
   <!-- <self_collide>true</self_collide> -->
 </gazebo>
@@ -29,13 +29,14 @@
   <self_collide>true</self_collide>
 </gazebo>
-<gazebo reference="lidar_1">
+<gazebo reference="lidar">
   <material>Gazebo/Black</material>
-  <sensor name="laser" type="ray">
+  <sensor name="laser" type="gpu_lidar">
+    <material>Gazebo/Black</material>
       <pose> 0 0 0 0 0 0 </pose>
       <visualize>false</visualize>
-      <always_on>true</always_on>
-      <enable_processing>true</enable_processing>
+      <!-- <always_on>true</always_on> -->
+      <!-- <enable_processing>true</enable_processing> -->
       <update_rate>10</update_rate>
-      <ray>
+      <lidar>
           <scan>
               <horizontal>
@@ -49,20 +50,17 @@
               <max>12</max>
           </range>
-      </ray>
-      <plugin name="laser_controller" filename="libgazebo_ros_ray_sensor.so">
-        <ros>
-          <argument>~/out:=scan</argument>
-      </ros>
-      <output_type>sensor_msgs/LaserScan</output_type>
-      <frame_name>lidar_1</frame_name>
-      </plugin>
+      </lidar>
+          <topic>scan</topic>
+          <gz_frame_id>lidar</gz_frame_id>
   </sensor>
 </gazebo>
 <gazebo reference="camera_1">
+  <material>Gazebo/Black</material>
     <sensor type="camera" name="camera">
         <pose> 0 0 0 0 0 0 </pose>
-        <visualize>false</visualize>
-        <update_rate>0.0</update_rate>
+        <visualize>true</visualize>
+        <update_rate>30.0</update_rate>
         <camera name="head">
+          <camera_info_topic>camera/camera_info</camera_info_topic>
           <horizontal_fov>1.089</horizontal_fov>
           <image>
@@ -76,12 +74,6 @@
           </clip>
         </camera>
-        <plugin name="camera_controller" filename="libgazebo_ros_camera.so">
-          <!-- <alwaysOn>true</alwaysOn>
-          <update_rate>0.0</update_rate> -->
-          <!-- <cameraName>mircobot/camera_optical</cameraName>
-          <imageTopicName>image_raw</imageTopicName>
-          <cameraInfoTopicName>camera_info</cameraInfoTopicName> -->
-          <frame_name>camera_optical</frame_name>
-        </plugin>
+        <topic>camera/image_raw</topic>
+        <gz_frame_id>camera_optical</gz_frame_id>
     </sensor>
 </gazebo>

File: mircobot_description/urdf/ros2_control.xacro (robot description, xacro)
@@ -3,7 +3,7 @@
     <ros2_control name="GazeboSystem" type="system">
         <hardware>
-            <plugin>gazebo_ros2_control/GazeboSystem</plugin>
+            <plugin>gz_ros2_control/GazeboSimSystem</plugin>
         </hardware>
-        <!-- <joint name="wheel_front_left_joint">
+        <joint name="wheel_front_left_joint">
             <command_interface name="velocity">
                 <param name="min">-10</param>
@@ -12,5 +12,5 @@
             <state_interface name="velocity"/>
             <state_interface name="position"/>
-        </joint> -->
+        </joint>
         <joint name="wheel_back_left_joint">
             <command_interface name="velocity">
@@ -21,5 +21,5 @@
             <state_interface name="position"/>
         </joint>
-        <!-- <joint name="wheel_front_right_joint">
+        <joint name="wheel_front_right_joint">
             <command_interface name="velocity">
                 <param name="min">-10</param>
@@ -28,5 +28,5 @@
             <state_interface name="velocity"/>
             <state_interface name="position"/>
-        </joint> -->
+        </joint>
         <joint name="wheel_back_right_joint">
             <command_interface name="velocity">
@@ -39,6 +39,7 @@
     </ros2_control>
     <gazebo>
-        <plugin name="gazebo_ros2_control" filename="libgazebo_ros2_control.so">
+         <plugin filename="gz_ros2_control-system" name="gz_ros2_control::GazeboSimROS2ControlPlugin">
             <parameters>$(find mircobot_description)/config/my_controllers.yaml</parameters>
+            <parameters>$(find mircobot_description)/config/gaz_ros2_ctl_use_sim.yaml</parameters>
         </plugin>
     </gazebo>
