Commit message: feat: migrate to ROS 2 Jazzy, add 3D Lidar and ros2_control

File: mircobot_description/urdf/mircobot.urdf.xacro (robot description, xacro)
@@ -2,4 +2,5 @@
 <robot name="mircobot" xmlns:xacro="http://www.ros.org/wiki/xacro">
     <xacro:arg name="use_ros2_control" default="true"/>
+    <xacro:arg name="use_mock_hardware" default="false"/>
     <xacro:include filename="$(find mircobot_description)/urdf/materials.xacro" />
     <!-- <xacro:include filename="$(find mircobot_description)/urdf/mircobot.trans" /> -->

File: mircobot_description/urdf/mircobot.xacro (robot description, xacro)
@@ -1,4 +1,10 @@
 <?xml version="1.0" ?>
 <robot name="mircobot" xmlns:xacro="http://www.ros.org/wiki/xacro">
+<link name="base_footprint"/>
+<joint name="base_footprint_joint" type="fixed">
+    <parent link="base_footprint"/>
+    <child link="base_link"/>
+    <origin xyz="0 0 0" rpy="0 0 0"/>
+</joint>
 <link name="base_link">
   <inertial>
@@ -20,12 +26,4 @@
     </geometry>
   </collision>
-</link>
-    <!-- BASE_FOOTPRINT LINK -->
-<joint name="base_footprint_joint" type="fixed">
-    <parent link="base_link"/>
-    <child link="base_footprint"/>
-    <origin xyz="0 0 0" rpy="0 0 0"/>
-</joint>
-<link name="base_footprint">
 </link>
 <joint name="wheel_front_left_joint" type="continuous">

File: mircobot_description/urdf/mircobot_gazebo.xacro (robot description, xacro)
@@ -45,4 +45,10 @@
                   <max_angle>3.14</max_angle>
               </horizontal>
+              <!-- 3D Lidar Vertical Scan (16 channels) -->
+              <vertical>
+                  <samples>16</samples>
+                  <min_angle>-0.26</min_angle>
+                  <max_angle>0.26</max_angle>
+              </vertical>
           </scan>
           <range>
@@ -51,5 +57,5 @@
           </range>
       </lidar>
-          <topic>scan</topic>
+          <topic>pointcloud</topic>
           <gz_frame_id>lidar</gz_frame_id>
   </sensor>

File: mircobot_description/urdf/ros2_control.xacro (robot description, xacro)
@@ -3,5 +3,10 @@
     <ros2_control name="GazeboSystem" type="system">
         <hardware>
-            <plugin>gz_ros2_control/GazeboSimSystem</plugin>
+            <xacro:if value="$(arg use_mock_hardware)">
+                <plugin>mock_components/GenericSystem</plugin>
+            </xacro:if>
+            <xacro:unless value="$(arg use_mock_hardware)">
+                <plugin>gz_ros2_control/GazeboSimSystem</plugin>
+            </xacro:unless>
         </hardware>
         <joint name="wheel_front_left_joint">
