Commit message: feat: warehouse env with isaacsim

File: mircobot_description/urdf/mircobot.urdf (robot description, URDF)
Before this commit: robot mircobot, 9 links, 8 joints
Links:
- removed link lidar_1
- added link lidar, mass 0.6042068071016569; collision mesh filename=../meshes/lidar_1.stl scale=0.001 0.001 0.001; visual mesh filename=../meshes/lidar_1.stl scale=0.001 0.001 0.001
- link base_link: geometry collision mesh filename=../meshes/base_link.stl scale=0.001 0.001 0.001; visual mesh filename=../meshes/base_link.stl scale=0.001 0.001 0.001
- link camera_1: geometry collision mesh filename=../meshes/camera_1.stl scale=0.001 0.001 0.001; visual mesh filename=../meshes/camera_1.stl scale=0.001 0.001 0.001
- link wheel_back_left_1: geometry collision mesh filename=../meshes/wheel_back_left_1.stl scale=0.001 0.001 0.001; visual mesh filename=../meshes/wheel_back_left_1.stl scale=0.001 0.001 0.001
- link wheel_back_right_1: geometry collision mesh filename=../meshes/wheel_back_right_1.stl scale=0.001 0.001 0.001; visual mesh filename=../meshes/wheel_back_right_1.stl scale=0.001 0.001 0.001
- link wheel_front_left_1: geometry collision mesh filename=../meshes/wheel_front_left_1.stl scale=0.001 0.001 0.001; visual mesh filename=../meshes/wheel_front_left_1.stl scale=0.001 0.001 0.001
- link wheel_front_right_1: geometry collision mesh filename=../meshes/wheel_front_right_1.stl scale=0.001 0.001 0.001; visual mesh filename=../meshes/wheel_front_right_1.stl scale=0.001 0.001 0.001
Joints:
- joint base_footprint_joint: child base_footprint -> base_link; parent base_link -> base_footprint
- joint lidar_joint: child lidar_1 -> lidar
- joint wheel_front_left_joint: type fixed -> continuous
- joint wheel_front_right_joint: type fixed -> continuous
